File: pcbs/amyboardr3.brd (EAGLE design)
At the start: 100 x 80 mm, 97 parts, among them M13 M2.5, M14 M2.5, M15 M2.5, M16 M2.5, Q2 S8050, Q5 S8050, SW2 JS102011JAQN, U1 PCM9211PT, U13 HX3608, U14 CH340K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

Commit message: .
Parts:
- removed 5V1, GND87: (no value), Discrete-new:TP-D45MIL
- removed VPWR1: (no value), Discrete:TP_4545
- added SPI: (no value), SparkFun-Connectors:1X06
Connections:
- removed net G: SPDIFIN.G, SPDIFOUT.G
- removed net IO11/MIDI_OUT: R90.1, U2.19
- removed net IO12/MIDI_IN: R91.2, U15.4, U2.20
- removed net IO13: U2.21
- removed net IO14: U2.22
- removed net IO17/I2C_SDA: I2C1.2
- removed net IO18/I2C_SCL: I2C1.1
- removed net IO21: U2.23
- removed net IO3: U2.15
- removed net IO4: U2.4
- removed net IO6: U2.6
- removed net IO7: U2.7
- new net AMY_FOLLOWER_SCL: I2C1.1, U2.5
- new net AMY_FOLLOWER_SDA: I2C1.2, U2.4
- new net MIDI_IN: R91.2, U15.4, U2.23
- new net MIDI_OUT: R90.1, U2.22
- new net SPI0_CS0: SPI.4, U2.18
- new net SPI0_MISO: SPI.2, U2.21
- new net SPI0_MOSI: SPI.3, U2.19
- new net SPI0_SCK: SPI.1, U2.20
- net +3V3: now also SPI.6
- net 5V: no longer 5V1.T
- net AMYOUT: now also U2.6; no longer U2.5
- net GND: now also SPDIFIN.G, SPDIFIN.S, SPDIFOUT.G, SPDIFOUT.S, SPI.5; no longer GND87.T, SPDIFOUT.T
- net GNDRX: no longer SPDIFIN.T
- net MCLK: now also U2.15, U2.7; no longer U2.18
- net SPDIFIN_SIGNAL: now also SPDIFIN.T; no longer SPDIFIN.S
- net SPDIFOUT_SIGNAL: now also SPDIFOUT.T; no longer SPDIFOUT.S
- net VPWR: no longer VPWR1.T
