File: pcbs/amyboardr3.sch (EAGLE design)
At the start: 79 parts, among them M13 M2.5, M14 M2.5, M15 M2.5, M16 M2.5, Q2 S8050, Q5 S8050, SW2 JS102011JAQN, U1 PCM9211PT, U14 CH340K, U15 H11L1SR2M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

Commit message: r3
Parts:
- removed AUDIO_CONN1, AUDIO_CONN2: 19269, microbuilder:AUDIO_3.5MMJACK
- removed R75, R76, R77: 0R, Discrete:R-0603
- removed R86: NC, Discrete:R-0603
- added 5V1, GND87: (no value), Discrete-new:TEST-POINT'4545'
- added AUDIO_INPUT, AUDIO_OUTPUT: 19269, microbuilder:AUDIO_3.5MMJACK
- added C1, C4: 0.1uF, Discrete-new:CAP-0603
- added C109: 22uF, Discrete-new:CAP-0603
- added C110: 100nF, Discrete-new:CAP-0603
- added C111: 22pF, Discrete-new:CAP-0603
- added C2, C3: 10uF, microbuilder:CAP_ELECTROLYTICPANASONIC_C
- added D15: SS54, diode:DIODE-DO-214AC
- added L4: 3.3µH/±30%/3.4A, SparkFun-Coils:INDUCTOR-CR54-3.3UH
- added R1, R2: 10K, adafruit:R-US_R0805
- added R3: 150, A9G:DISCRETE_R-0603
- added R93: 100K, A9G:DISCRETE_R-0603
- added R94, R95: NC, A9G:DISCRETE_R-0603
- added R96: 0R, A9G:DISCRETE_R-0603
- added R97: 88.7K, A9G:DISCRETE_R-0603
- added R98: 12K, A9G:DISCRETE_R-0603
- added U13: HX3608, self:HX3608
- added Y1: ABM10W-22.5792MHZ-8-K1Z-T3, ABM10W-22.5792MHZ-8-K1Z-T3:ABM10W-22.5792MHZ-8-K1Z-T3
Connections:
- removed net DIN: PCM5101.DIN, R75.2
- removed net IO10: U2.IO10
- removed net IO18/I2C_SCL1: R86.1, U2.IO18
- removed net IO2: R77.1, U2.IO2
- removed net IO5: R75.1, U2.IO5
- removed net IO8: R76.1, U2.IO8
- removed net IO9: U2.IO9
- new net AMYIN: U1.DOUT, U2.IO9
- new net AMYOUT: PCM5101.DIN, U1.MPIO_C3, U2.IO5
- new net ENABLE: R93.1, U13.EN
- new net GNDRX: SPDIFIN.T, U1.GNDRX
- new net I2C_SCL: U1.MC/SCL, U2.IO18
- new net I2C_SDA: U1.MDL/SDA, U2.IO17
- new net LINX: R2.2, U1.VINL
- new net MCLK: U1.MPIO_CO, U1.SCKO, U2.IO10
- new net N$1: C1.2, U1.RXINO
- new net N$2: C4.2, R3.2
- new net N$3: C4.1, U1.MPOO
- new net N$4: C2.+, R2.1
- new net N$5: C3.+, R1.2
- new net N$65: D15.A, L4.2, U13.SW
- new net N$66: C111.2, R97.1, R98.2, U13.FB
- new net N$67: R94.2, U13.NC
- new net N$68: R95.1, R96.1, U13.VIN
- new net RINX: R1.1, U1.VINR
- new net SPDIFIN_SIGNAL: C1.1, SPDIFIN.S
- new net SPDIFOUT_SIGNAL: R3.1, SPDIFOUT.S
- new net XTI: U1.XTI, Y1.1
- new net XTO: U1.XTO, Y1.2
- net +3V3: now also U1.DVDD, U1.RST, U1.VCC, U1.VDDRX; no longer R86.2
- net 5V: now also 5V1.T, C109.1, C110.1, C111.1, D15.C, R96.2, R97.2, U1.VCCAD
- net AGND: now also AUDIO_INPUT.P$1, AUDIO_OUTPUT.P$1, U1.AGND, U1.AGNDAD; no longer AUDIO_CONN1.P$1, AUDIO_CONN2.P$1
- net BCLK: now also U1.BCK, U1.MPIO_C1, U2.IO8; no longer R76.2
- net GND: now also C109.2, C110.2, GND87.T, R94.1, R98.1, SPDIFOUT.T, U1.DGND, U1.MDO/ADRO, U1.MODE, U1.MS/ADR1, U13.GND, Y1.GND
- net IO17/I2C_SDA: no longer U2.IO17
- net LIN: now also AUDIO_INPUT.P$4, AUDIO_INPUT.P$5, C2.-; no longer AUDIO_CONN1.P$4, AUDIO_CONN1.P$5
- net LOUT: now also AUDIO_OUTPUT.P$4, AUDIO_OUTPUT.P$5; no longer AUDIO_CONN2.P$4, AUDIO_CONN2.P$5
- net LRC: now also U1.LRCK, U1.MPIO_C2, U2.IO2; no longer R77.2
- net RIN: now also AUDIO_INPUT.P$2, AUDIO_INPUT.P$3, C3.-; no longer AUDIO_CONN1.P$2, AUDIO_CONN1.P$3
- net ROUT: now also AUDIO_OUTPUT.P$2, AUDIO_OUTPUT.P$3; no longer AUDIO_CONN2.P$2, AUDIO_CONN2.P$3
- net VPWR: now also L4.1, R93.2, R95.2
Other:
- note added: "2A"
- note added: "3v3->5V boost"
- note added: "DAC and ADC and MIDI"
- note added: "ESP32S3"
- note added: "Fb=0.6V"
- note added: "PCM9211"
- moved on the sheet: C101, C102, C103, D13, I2C1, M13, M14, M15, M16, MIDI_IN_CONN1, MIDI_OUT_CONN1, Q2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

Commit message: .
Parts:
- removed 5V1, GND87: (no value), Discrete-new:TEST-POINT'4545'
- removed VPWR1: (no value), Discrete:PAD-TEST-POINT-CIRCLE'4545'
- added SPI: (no value), SparkFun-Connectors:CONN_06SILK_FEMALE_PTH
Connections:
- removed net IO11/MIDI_OUT: R90.1, U2.IO11
- removed net IO12/MIDI_IN: R91.2, U15.VO, U2.IO12
- removed net IO13: U2.IO13
- removed net IO14: U2.IO14
- removed net IO17/I2C_SDA: I2C1.2
- removed net IO18/I2C_SCL: I2C1.1
- removed net IO21: U2.IO21
- removed net IO3: U2.IO3
- removed net IO4: U2.IO4
- removed net IO6: U2.IO6
- removed net IO7: U2.IO7
- new net AMY_FOLLOWER_SCL: I2C1.1, U2.IO5
- new net AMY_FOLLOWER_SDA: I2C1.2, U2.IO4
- new net MIDI_IN: R91.2, U15.VO, U2.IO21
- new net MIDI_OUT: R90.1, U2.IO14
- new net SPI0_CS0: SPI.4, U2.IO10
- new net SPI0_MISO: SPI.2, U2.IO13
- new net SPI0_MOSI: SPI.3, U2.IO11
- new net SPI0_SCK: SPI.1, U2.IO12
- net +3V3: now also SPI.6
- net 5V: no longer 5V1.T
- net AMYOUT: now also U2.IO6; no longer U2.IO5
- net GND: now also SPDIFIN.G, SPDIFIN.S, SPDIFOUT.G, SPDIFOUT.S, SPI.5; no longer GND87.T, SPDIFOUT.T
- net GNDRX: no longer SPDIFIN.T
- net MCLK: now also U2.IO3, U2.IO7; no longer U2.IO10
- net SPDIFIN_SIGNAL: now also SPDIFIN.T; no longer SPDIFIN.S
- net SPDIFOUT_SIGNAL: now also SPDIFOUT.T; no longer SPDIFOUT.S
- net VPWR: no longer VPWR1.T
Other:
- note added: "HEADERS"
- note added: "NOTES/TODO: - RXGND? Is it just GND? - CV jacks using ADC / DACs on ESP? Or DAC i2c module? - Expanded header with 5V, extra GPIOs - GND unused pins?? - Put in dan's board changes & XTAL circuit - Confirm power / VPWR / 3v3 / 5v - Move SPDIF to 3.5mm jacks, confirm RCA pins are right"
- note added: "USB, UART"
- note removed: "USB to UART"
- moved on the sheet: AUDIO_INPUT, AUDIO_OUTPUT, C100, C101, C102, C103, C104, C105, C106, C107, C108, C109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
