File: pcbs/amyboardr3.sch (EAGLE design)
At the start: 109 parts, among them M13 M2.5, M14 M2.5, M15 M2.5, M16 M2.5, Q2 S8050, Q5 S8050, SW2 JS102011JAQN, U1 PCM9211PT, U13 HX3608, U14 CH340K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

Commit message: caps
Parts:
- removed C10, C9: 10 pf, capacitor-wima:C-2.5-5/4
- added C18, C19: 10pF, Discrete-new:CAP-0603
Connections:
- net GND: now also C18.2, C19.2; no longer C10.2, C9.2
- net XTI: now also C19.1; no longer C9.1
- net XTO: now also C18.1; no longer C10.1
Changed lines of the file:
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@@
 <part name="C7" library="microbuilder" deviceset="CAP_ELECTROLYTIC" device="PANASONIC_C" value="10uF"/>
 <part name="C5" library="microbuilder" deviceset="CAP_CERAMIC" device="0805-NOOUTLINE" value="0.1uF"/>
-<part name="C9" library="capacitor-wima" library_urn="urn:adsk.eagle:library:116" deviceset="C-" device="2.5-5/4" package3d_urn="urn:adsk.eagle:package:5439/1" value="10 pf"/>
-<part name="C10" library="capacitor-wima" library_urn="urn:adsk.eagle:library:116" deviceset="C-" device="2.5-5/4" package3d_urn="urn:adsk.eagle:package:5439/1" value="10 pf"/>
 <part name="C11" library="microbuilder" deviceset="CAP_CERAMIC" device="0805-NOOUTLINE" value="0.1uF"/>
 <part name="C12" library="microbuilder" deviceset="CAP_ELECTROLYTIC" device="PANASONIC_C" value="10uF"/>
@@
 <part name="C17" library="microbuilder" deviceset="CAP_CERAMIC" device="0805-NOOUTLINE" value="4.7nF"/>
 <part name="R4" library="adafruit" deviceset="R-US_" device="R0805" value="680"/>
+<part name="C18" library="Discrete-new" deviceset="CAP" device="-0603" value="10pF"/>
+<part name="C19" library="Discrete-new" deviceset="CAP" device="-0603" value="10pF"/>
 </parts>
 <sheets>
@@
 <attribute name="VALUE" x="108.98" y="158.73" size="1.27" layer="96" font="vector" rot="R90"/>
 </instance>
-<instance part="C9" gate="G$1" x="5.08" y="-38.1" smashed="yes">
-<attribute name="NAME" x="6.604" y="-37.719" size="1.778" layer="95"/>
-<attribute name="VALUE" x="6.604" y="-42.799" size="1.778" layer="96"/>
-</instance>
-<instance part="C10" gate="G$1" x="33.02" y="-38.1" smashed="yes">
-<attribute name="NAME" x="34.544" y="-37.719" size="1.778" layer="95"/>
-<attribute name="VALUE" x="34.544" y="-42.799" size="1.778" layer="96"/>
-</instance>
 <instance part="C11" gate="G$1" x="91.44" y="149.86" smashed="yes">
 <attribute name="NAME" x="89.15" y="151.11" size="1.27" layer="95" font="vector" rot="R90"/>
@@
 <attribute name="NAME" x="-11.43" y="82.042" size="1.27" layer="95" font="vector" rot="R90"/>
 <attribute name="VALUE" x="-7.874" y="82.042" size="1.016" layer="96" font="vector" ratio="15" rot="R90"/>
+</instance>
+<instance part="C18" gate="C" x="33.02" y="-39.37" smashed="yes" rot="R270">
+<attribute name="NAME" x="29.464" y="-38.354" size="1.27" layer="95" ratio="10"/>
+<attribute name="VALUE" x="27.178" y="-41.656" size="1.27" layer="96" ratio="10"/>
+</instance>
+<instance part="C19" gate="C" x="5.08" y="-39.37" smashed="yes" rot="R270">
+<attribute name="NAME" x="1.524" y="-38.354" size="1.27" layer="95" ratio="10"/>
+<attribute name="VALUE" x="-0.762" y="-41.656" size="1.27" layer="96" ratio="10"/>
 </instance>
 </instances>
@@
 </segment>
 <segment>
-<pinref part="C9" gate="G$1" pin="2"/>
 <wire x1="5.08" y1="-43.18" x2="5.08" y2="-45.72" width="0.1524" layer="91"/>
 <label x="5.08" y="-45.72" size="1.778" layer="95"/>
+<pinref part="C19" gate="C" pin="2"/>
 </segment>
 <segment>
@@
 <pinref part="Y1" gate="G$1" pin="GND"/>
 <wire x1="27.94" y1="-40.64" x2="27.94" y2="-43.18" width="0.1524" layer="91"/>
-<pinref part="C10" gate="G$1" pin="2"/>
 <wire x1="27.94" y1="-43.18" x2="33.02" y2="-43.18" width="0.1524" layer="91"/>
+<label x="43.18" y="-43.18" size="1.778" layer="95"/>
+<pinref part="C18" gate="C" pin="2"/>
 <wire x1="33.02" y1="-43.18" x2="43.18" y2="-43.18" width="0.1524" layer="91"/>
 <junction x="33.02" y="-43.18"/>
-<label x="43.18" y="-43.18" size="1.778" layer="95"/>
 </segment>
 <segment>
@@
 <wire x1="12.7" y1="-35.56" x2="5.08" y2="-35.56" width="0.1524" layer="91"/>
 <label x="2.54" y="-35.56" size="1.778" layer="95"/>
-<pinref part="C9" gate="G$1" pin="1"/>
+<pinref part="C19" gate="C" pin="1"/>
 <wire x1="5.08" y1="-35.56" x2="0" y2="-35.56" width="0.1524" layer="91"/>
 <junction x="5.08" y="-35.56"/>
@@
 <segment>
 <pinref part="Y1" gate="G$1" pin="2"/>
+<label x="35.56" y="-35.56" size="1.778" layer="95"/>
 <wire x1="27.94" y1="-35.56" x2="33.02" y2="-35.56" width="0.1524" layer="91"/>
-<label x="35.56" y="-35.56" size="1.778" layer="95"/>
-<pinref part="C10" gate="G$1" pin="1"/>
+<pinref part="C18" gate="C" pin="1"/>
 <wire x1="33.02" y1="-35.56" x2="40.64" y2="-35.56" width="0.1524" layer="91"/>
 <junction x="33.02" y="-35.56"/>

Commit message: moving to 3.5mm jacks for everything
Parts:
- removed AUDIO_INPUT: 19269, microbuilder:AUDIO_3.5MMJACK
- removed SPDIFIN, SPDIFOUT: PJRAS1X1S01, PJRAS1X1S01:PJRAS1X1S01
- added J11, J12, J13, J14, J15, J16, J17, J18, J19, J20: SJ1-3543, SJ1-3543:SJ1-3543
Connections:
- net AGND: now also J11.1; no longer AUDIO_INPUT.P$1
- net BCLK: now also J20.2
- net GND: no longer SPDIFIN.G, SPDIFIN.S, SPDIFOUT.G, SPDIFOUT.S
- net LIN: now also J11.2; no longer AUDIO_INPUT.P$4, AUDIO_INPUT.P$5
- net LINX: now also J20.1
- net RIN: now also J11.3; no longer AUDIO_INPUT.P$2, AUDIO_INPUT.P$3
- net RINX: now also J20.3
- net SPDIFIN_SIGNAL: no longer SPDIFIN.T
- net SPDIFOUT_SIGNAL: no longer SPDIFOUT.T

Commit message: stacked audio jacks
Parts:
- removed AUDIO_OUTPUT, MIDI_IN_CONN1, MIDI_OUT_CONN1: 19269, microbuilder:AUDIO_3.5MMJACK
- removed J12, J13, J14, J15, J16, J17, J18, J19, J20: SJ1-3543, SJ1-3543:SJ1-3543
- added CV_IN1, CV_IN2, CV_OUT1, CV_OUT2, LINE_OUT, MIDI_IN, MIDI_OUT, SPDIF_IN, SPDIF_OUT: SJ1-3543, SJ1-3543:SJ1-3543
- added U$1, U$2, U$3, U$4, U$5, U$6: NC_MARKER, NC_MARKER:NC_MARKER
- renumbered J11 to LINE_IN
Connections:
- removed net IO15: U2.IO15
- removed net IO16: U2.IO16
- removed net IO38: U2.IO38
- removed net IO39: U2.IO39
- new net ADC0: CV_IN2.2, U2.IO15
- new net ADC1: CV_IN1.2, U2.IO16
- new net N$10: SPDIF_IN.3, U$2.P$1
- new net N$11: CV_OUT1.3, U$3.P$1
- new net N$12: CV_OUT2.3, U$4.P$1
- new net N$13: CV_IN1.3, U$5.P$1
- new net N$14: CV_IN2.3, U$6.P$1
- new net N$9: SPDIF_OUT.3, U$1.P$1
- new net PWM0: CV_OUT1.2, U2.IO38
- new net PWM1: CV_OUT2.2, U2.IO39
- net AGND: now also LINE_OUT.1; no longer AUDIO_OUTPUT.P$1
- net BCLK: no longer J20.2
- net GND: now also CV_IN1.1, CV_IN2.1, CV_OUT1.1, CV_OUT2.1, MIDI_IN.1, MIDI_OUT.1, SPDIF_IN.1, SPDIF_OUT.1; no longer MIDI_IN_CONN1.P$1, MIDI_OUT_CONN1.P$1
- net LINX: no longer J20.1
- net LOUT: now also LINE_OUT.2; no longer AUDIO_OUTPUT.P$4, AUDIO_OUTPUT.P$5
- net N$55: now also MIDI_IN.2; no longer MIDI_IN_CONN1.P$4, MIDI_IN_CONN1.P$5
- net N$56: now also MIDI_IN.3; no longer MIDI_IN_CONN1.P$2, MIDI_IN_CONN1.P$3
- net N$58: now also MIDI_OUT.2; no longer MIDI_OUT_CONN1.P$4, MIDI_OUT_CONN1.P$5
- net N$59: now also MIDI_OUT.3; no longer MIDI_OUT_CONN1.P$2, MIDI_OUT_CONN1.P$3
- net RINX: no longer J20.3
- net ROUT: now also LINE_OUT.3; no longer AUDIO_OUTPUT.P$2, AUDIO_OUTPUT.P$3
- net SPDIFIN_SIGNAL: now also SPDIF_IN.2
- net SPDIFOUT_SIGNAL: now also SPDIF_OUT.2
Other:
- note added: "NOTES/TODO: - RXGND? Is it just GND? - Transistor for CVOUTs to 0-10V from 3.3V - Voltage divider for CVIns to 3.3V from 0-10V - Expanded header with 5V, extra GPIOs, UART - I2C main grove/mabee connector as well - NC/GND unused pins - Confirm power / VPWR / 3v3 / 5v"
- note removed: "NOTES/TODO: - RXGND? Is it just GND? - CV jacks using ADC / DACs on ESP? Or DAC i2c module? - Expanded header with 5V, extra GPIOs - GND unused pins?? - Put in dan's board changes & XTAL circuit - Confirm power / VPWR / 3v3 / 5v - Move SPDIF to 3.5mm jacks, confirm RCA pins are right"

Commit message: dac/adcs
Parts:
- added C10, C9: 10nF, Discrete-new:CAP-0603
- added MABEEDAC: (no value), SparkFun-Connectors:CONN_04
- added R5, R7: 68K, adafruit:R-US_R0805
- added R6, R8: 33K, adafruit:R-US_R0805
Connections:
- new net MABEEDAC_VOUT0: CV_OUT1.2, MABEEDAC.3
- new net MABEEDAC_VOUT1: CV_OUT2.2, MABEEDAC.4
- new net N$15: CV_OUT2.1
- new net N$16: C9.1, CV_IN2.2, R7.2, R8.1
- new net N$18: C10.1, CV_IN1.2, R5.2, R6.1
- net +3V3: now also MABEEDAC.2
- net ADC0: now also R5.1; no longer CV_IN2.2
- net ADC1: now also R7.1; no longer CV_IN1.2
- net GND: now also C10.2, C9.2, MABEEDAC.1, R6.2, R8.2; no longer CV_OUT2.1
- net PWM0: no longer CV_OUT1.2
- net PWM1: no longer CV_OUT2.2
Other:
- note added: "NOTES/TODO: - RXGND? Is it just GND? - MabeeDAC to provide VOUT0 and VOUT1 - Expanded header with 5V, extra GPIOs, UART - I2C main grove/mabee connector as well ?? - NC/GND unused pins - Confirm power / VPWR / 3v3 / 5v - Remove/test single USB NATIVE port"
- note removed: "NOTES/TODO: - RXGND? Is it just GND? - Transistor for CVOUTs to 0-10V from 3.3V - Voltage divider for CVIns to 3.3V from 0-10V - Expanded header with 5V, extra GPIOs, UART - I2C main grove/mabee connector as well - NC/GND unused pins - Confirm power / VPWR / 3v3 / 5v"
- moved on the sheet: CV_IN1, CV_IN2

Commit message: header, fixed adcs
Parts:
- added J1: 52601-G10-8LF, 52601-G10-8LF:52601-G10-8LF
- C10, C9: value 10nF -> 1nF
Connections:
- removed net N$16: C9.1, CV_IN2.2, R7.2, R8.1
- removed net N$18: C10.1, CV_IN1.2, R5.2, R6.1
- new net +12V: J1.09, J1.10
- new net -12V: J1.01, J1.02
- new net N$17: CV_IN1.2, R5.1
- new net N$19: CV_IN2.2, R7.1
- net ADC0: now also C10.1, R5.2, R6.1; no longer R5.1
- net ADC1: now also C9.1, R7.2, R8.1; no longer R7.1
- net GND: now also J1.03, J1.04, J1.05, J1.06, J1.07, J1.08
Other:
- moved on the sheet: C10, C9, CV_IN1, CV_IN2, MABEEDAC, R5, R6, R7, R8
