File: pcbs/amyboardr4.sch (EAGLE design)
At the start: 165 parts, among them J1 52601-G10-8LF, Q2 S8050, Q5 S8050, U1 PCM9211PT, U13 HX3608, U15 H11L1SR2M, U16 SPX3819, U2 ESP32­S2­SOLO, U4 TL074CD, U6 HX3608, Y1 22.5792MHZ

Commit message: 4 way DIN, VPWR
Parts:
- removed C101, C104: 10uF, Discrete:C-0603
- removed C102: 0.1uF, A9G:DISCRETE_C-0603
- removed C105: 10uF, A9G:DISCRETE_C-0603
- removed C109: 22uF, Discrete-new:CAP-0603
- removed C110: 100nF, Discrete-new:CAP-0603
- removed C111: 22pF, Discrete-new:CAP-0603
- removed D15: SS54, diode:DIODE-DO-214AC
- removed L4: 3.3µH/±30%/3.4A, SparkFun-Coils:INDUCTOR-CR54-3.3UH
- removed R23, R24: 10K, adafruit:R-US_R0805
- removed R92: 0R, Discrete:R-0603
- removed R93: 100K, A9G:DISCRETE_R-0603
- removed R94, R95: NC, A9G:DISCRETE_R-0603
- removed R96: 0R, A9G:DISCRETE_R-0603
- removed R97: 88.7K, A9G:DISCRETE_R-0603
- removed R98: 12K, A9G:DISCRETE_R-0603
- removed S1: SWS008, smd-special:SWS008
- removed U13: HX3608, self:HX3608
- added 1-10VPP: 218-4LPSTR, 218-4LPSTR:218-4LPSTR
- added C35: NC, Discrete:C-0603
- added D1, D2: SS54, diode:DIODE-DO-214AC
- added U3: SPX3819, IC:SPX3819
- C32: value 10uF -> 4.7uF/16V; device microbuilder:CAP_ELECTROLYTICPANASONIC_C -> Discrete:C-0603
- C33: value 0.1uF -> 10uF; device microbuilder:CAP_CERAMIC0805-NOOUTLINE -> Discrete:C-0603
Connections:
- net VBUS renamed 5V_IN
- removed net N$16: R5.2, R6.1, S1.8
- removed net N$30: R23.1, S1.6
- removed net N$32: R24.1, S1.5
- removed net N$65: D15.A, L4.2, U13.SW
- removed net N$66: C111.2, R97.1, R98.2, U13.FB
- removed net N$67: R94.2, U13.NC
- removed net N$68: R95.1, R96.1, U13.VIN
- new net 12V_IN: D2.A, J1.09, J1.10
- new net 3V3_IN: D1.A, I2C_CONTROL.3
- net +12V: no longer J1.09, J1.10
- net +3V3: no longer C105.2, C32.+, C33.1, I2C_CONTROL.3, R23.2, R24.2, R92.1
- net -12V: no longer J1.01, J1.02
- net 3.3V: no longer C104.1, R92.2
- net 5V: now also C33.1, U3.VOUT; no longer C101.1, C102.2, C109.1, C110.1, C111.1, D14.C, D15.C, R96.2, R97.2
- net ADC1: now also R5.2, R6.1; no longer S1.9
- net ADC2: now also R20.2, R21.1; no longer S1.10
- net AGND: no longer C32.-, C33.2
- net ENABLE: no longer R93.1, U13.EN
- net GND: now also C32.2, C33.2, C35.2, J1.01, J1.02, U3.GND; no longer C101.2, C102.1, C104.2, C105.1, C109.2, C110.2, R94.1, R98.1, U13.GND
- net N$15: now also C35.1, U3.BYP; no longer R20.2, R21.1, S1.7
- net N$31: no longer S1.12
- net N$33: no longer S1.11
- net N$35: now also 1-10VPP.5; no longer S1.1
- net N$36: now also 1-10VPP.6; no longer S1.2
- net N$4: now also 1-10VPP.1; no longer S1.13
- net N$40: now also 1-10VPP.8; no longer S1.4
- net N$41: now also 1-10VPP.7; no longer S1.3
- net N$44: now also 1-10VPP.3; no longer S1.15
- net N$45: now also 1-10VPP.4; no longer S1.16
- net N$5: now also 1-10VPP.2; no longer S1.14
- net VPWR: now also C32.1, D1.C, D14.C, D2.C, U3.EN, U3.VIN; no longer L4.1, R93.2, R95.2
Other:
- note added: "ME6214C33"
- note added: "ME6214C50"
- note added: "NOTES/TODO: - NC/GND unused pins? - Confirm VPWR / 3v3 / 5v / 12V"
- note removed: "3v3->5V boost"
- note removed: "ME6217"
- note removed: "NOTES/TODO: - NC/GND unused pins - 12V -> 5V regulator for modular port - Confirm VOUT / VPWR / 3v3 / 5v / 12V"
- note removed: "POWER AND FILTERING"
- moved on the sheet: C2, C20, C27, C28, C29, C3, C30, C31, C34, C70, C85, D10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
