File: pcbs/amyboardr4.sch (EAGLE design)
At the start: 150 parts, among them J1 52601-G10-8LF, Q2 S8050, Q5 S8050, U1 PCM9211PT, U15 H11L1SR2M, U16 SPX3819, U2 ESP32­S2­SOLO, U3 SPX3819, U4 TL074CD, U6 HX3608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

Commit message: adding back in dan's r4
Parts:
- removed 1-10VPP: 218-4LPSTR, 218-4LPSTR:218-4LPSTR
- removed C35: NC, Discrete:C-0603
- removed D1, D2: SS54, diode:DIODE-DO-214AC
- removed U3: SPX3819, IC:SPX3819
- added C101, C104: 10uF, Discrete:C-0603
- added C102: 0.1uF, A9G:DISCRETE_C-0603
- added C105: 10uF, A9G:DISCRETE_C-0603
- added C109: 22uF, Discrete-new:CAP-0603
- added C110: 100nF, Discrete-new:CAP-0603
- added C111, C25: 22pF, Discrete-new:CAP-0603
- added D15: SS54, diode:DIODE-DO-214AC
- added D4, D5, D6: 1N5819HW-7-F, 1N5819HW-7-F:1N5819HW-7-F
- added L2: 1269AS-H-100N=P2, 1269AS-H-100N_P2:1269AS-H-100N=P2
- added L4: 3.3µH/±30%/3.4A, SparkFun-Coils:INDUCTOR-CR54-3.3UH
- added R12: 1M, A9G:DISCRETE_R-0603
- added R13: 115K, A9G:DISCRETE_R-0603
- added R23, R24: 10K, adafruit:R-US_R0805
- added R92: 0R, Discrete:R-0603
- added R93: 100K, A9G:DISCRETE_R-0603
- added R94, R95: NC, A9G:DISCRETE_R-0603
- added R96: 0R, A9G:DISCRETE_R-0603
- added R97: 88.7K, A9G:DISCRETE_R-0603
- added R98: 12K, A9G:DISCRETE_R-0603
- added S1: SWS008, smd-special:SWS008
- added U13: HX3608, self:HX3608
- added U5: TPS61040DBVR, TPS61040DBVR:TPS61040DBVR
- C32: value 4.7uF/16V -> 10uF; device Discrete:C-0603 -> microbuilder:CAP_ELECTROLYTICPANASONIC_C
- C33: value 10uF -> 0.1uF; device Discrete:C-0603 -> microbuilder:CAP_CERAMIC0805-NOOUTLINE
Connections:
- net 5V_IN renamed VBUS
- removed net 12V_IN: D2.A, J1.09, J1.10
- removed net 3V3_IN: D1.A, I2C_CONTROL.3
- new net N$16: R5.2, R6.1, S1.8
- new net N$23: D4.A, L2.1, U5.SW
- new net N$24: C25.1, D4.K, R12.2
- new net N$25: C25.2, R12.1, R13.2, U5.FB
- new net N$30: R23.1, S1.6
- new net N$32: R24.1, S1.5
- new net N$65: D15.A, L4.2, U13.SW
- new net N$66: C111.2, R97.1, R98.2, U13.FB
- new net N$67: R94.2, U13.NC
- new net N$68: R95.1, R96.1, U13.VIN
- net +12V: now also J1.09, J1.10
- net +3V3: now also C105.2, C32.+, C33.1, I2C_CONTROL.3, L2.2, R23.2, R24.2, R92.1, U5.EN, U5.VIN
- net -12V: now also J1.01, J1.02
- net 3.3V: now also C104.1, R92.2
- net 5V: now also C101.1, C102.2, C109.1, C110.1, C111.1, D14.C, D15.C, R96.2, R97.2; no longer C33.1, U3.VOUT
- net ADC1: now also S1.9; no longer R5.2, R6.1
- net ADC2: now also S1.10; no longer R20.2, R21.1
- net AGND: now also C32.-, C33.2
- net ENABLE: now also R93.1, U13.EN
- net GND: now also C101.2, C102.1, C104.2, C105.1, C109.2, C110.2, R13.1, R94.1, R98.1, U13.GND, U5.GND; no longer C32.2, C33.2, C35.2, J1.01, J1.02, U3.GND
- net N$15: now also R20.2, R21.1, S1.7; no longer C35.1, U3.BYP
- net N$31: now also S1.12
- net N$33: now also S1.11
- net N$35: now also S1.1; no longer 1-10VPP.5
- net N$36: now also S1.2; no longer 1-10VPP.6
- net N$4: now also S1.13; no longer 1-10VPP.1
- net N$40: now also S1.4; no longer 1-10VPP.8
- net N$41: now also S1.3; no longer 1-10VPP.7
- net N$44: now also S1.15; no longer 1-10VPP.3
- net N$45: now also S1.16; no longer 1-10VPP.4
- net N$5: now also S1.14; no longer 1-10VPP.2
- net VPWR: now also L4.1, R93.2, R95.2; no longer C32.1, D1.C, D14.C, D2.C, U3.EN, U3.VIN
Other:
- note added: "3v3->5V boost"
- note added: "ME6217"
- note added: "NOTES/TODO: - MabeeDAC to provide VOUT0 and VOUT1 - NC/GND unused pins - 12V -> 5V regulator for modular port - Confirm VOUT / VPWR / 3v3 / 5v / 12V"
- note added: "POWER AND FILTERING"
- note removed: "ME6214C33"
- note removed: "ME6214C50"
- note removed: "NOTES/TODO: - NC/GND unused pins? - Confirm VPWR / 3v3 / 5v / 12V"
- moved on the sheet: C2, C20, C27, C28, C29, C3, C30, C31, C34, C70, C85, D10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
