File: pcbs/amyboardr4.brd (EAGLE design)
At the start: 106.1 x 47.5 mm, 144 parts, among them J1 52601-G10-8LF, Q2 S8050, Q5 S8050, U1 PCM9211PT, U15 H11L1SR2M, U16 SPX3819, U2 ESP32­S2­SOLO, U3 SPX3819, U4 TL074CD, U6 HX3608, Y1 22.5792MHZ

Commit message: adding back in dan's r4
Parts:
- removed 1-10VPP: 218-4LPSTR, 218-4LPSTR:SW_218-4LPSTR
- removed C35: NC, Discrete:0603
- removed D1, D2: SS54, diode:DO-214AC
- removed U3: SPX3819, IC:SOT23-5
- added C101, C104: 10uF, Discrete:0603
- added C102: 0.1uF, A9G:DISCRETE_C0603
- added C105: 10uF, A9G:DISCRETE_C0603
- added C109: 22uF, Discrete-new:C0603
- added C110: 100nF, Discrete-new:C0603
- added C111, C25: 22pF, Discrete-new:C0603
- added D15: SS54, diode:DO-214AC
- added D4, D5, D6: 1N5819HW-7-F, 1N5819HW-7-F:SOD3715X145N
- added L2: 1269AS-H-100N=P2, 1269AS-H-100N_P2:INDC2520X100N
- added L4: 3.3µH/±30%/3.4A, SparkFun-Coils:CR54
- added R12: 1M, A9G:DISCRETE_R0603
- added R13: 115K, A9G:DISCRETE_R0603
- added R23, R24: 10K, adafruit:R0805
- added R92: 0R, Discrete:R0603
- added R93: 100K, A9G:DISCRETE_R0603
- added R94, R95: NC, A9G:DISCRETE_R0603
- added R96: 0R, A9G:DISCRETE_R0603
- added R97: 88.7K, A9G:DISCRETE_R0603
- added R98: 12K, A9G:DISCRETE_R0603
- added S1: SWS008, smd-special:SMS-008
- added U13: HX3608, self:SOT-23-6
- added U5: TPS61040DBVR, TPS61040DBVR:SOT95P280X145-5N
- C32: value 4.7uF/16V -> 10uF; device Discrete:0603 -> microbuilder:PANASONIC_C
- C33: value 10uF -> 0.1uF; device Discrete:0603 -> microbuilder:0805-NO@1
- moved R26 1320.6 mm to (-350.3, -1222.8)
- moved R28 1320.6 mm to (-350.3, -1234.4)
- moved C2 1320.6 mm to (-356.1, -1244.6)
- moved C3 1320.6 mm to (-363.2, -1244.6)
- moved R25 1320.6 mm to (-350.3, -1216.9)
- moved R27 1320.6 mm to (-350.3, -1228.6)
- moved R29 1320.6 mm to (-350.3, -1240.3)
- moved R30 1320.6 mm to (-350.3, -1246.1)
- moved C26 1242.6 mm to (-350.8, -1170.2)
- moved R10 1242.6 mm to (-350.3, -1174.5)
- moved R8 1242.6 mm to (-343.4, -1161.0)
- moved C22 1242.6 mm to (-349.0, -1159.5)
- moved C23 1242.6 mm to (-350.8, -1165.1)
- moved C24 1242.6 mm to (-350.8, -1167.6)
- moved R11 1242.6 mm to (-350.3, -1180.3)
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Connections:
- net 5V_IN renamed VBUS
- removed net 12V_IN: D2.A, J1.09, J1.10
- removed net 3V3_IN: D1.A, I2C_CONTROL.3
- new net N$16: R5.2, R6.1, S1.8
- new net N$23: D4.A, L2.1, U5.1
- new net N$24: C25.1, D4.C, R12.2
- new net N$25: C25.2, R12.1, R13.2, U5.3
- new net N$30: R23.1, S1.6
- new net N$32: R24.1, S1.5
- new net N$65: D15.A, L4.P$2, U13.1
- new net N$66: C111.2, R97.1, R98.2, U13.3
- new net N$67: R94.2, U13.6
- new net N$68: R95.1, R96.1, U13.5
- net +12V: now also J1.09, J1.10
- net +3V3: now also C105.2, C32.+, C33.1, I2C_CONTROL.3, L2.2, R23.2, R24.2, R92.1, U5.4, U5.5
- net -12V: now also J1.01, J1.02
- net 3.3V: now also C104.1, R92.2
- net 5V: now also C101.1, C102.2, C109.1, C110.1, C111.1, D14.C, D15.C, R96.2, R97.2; no longer C33.1, U3.5
- net ADC1: now also S1.9; no longer R5.2, R6.1
- net ADC2: now also S1.10; no longer R20.2, R21.1
- net AGND: now also C32.-, C33.2
- net ENABLE: now also R93.1, U13.4
- net GND: now also C101.2, C102.1, C104.2, C105.1, C109.2, C110.2, R13.1, R94.1, R98.1, U13.2, U5.2; no longer C32.2, C33.2, C35.2, J1.01, J1.02, U3.2
- net N$15: now also R20.2, R21.1, S1.7; no longer C35.1, U3.4
- net N$31: now also S1.12
- net N$33: now also S1.11
- net N$35: now also S1.1; no longer 1-10VPP.5
- net N$36: now also S1.2; no longer 1-10VPP.6
- net N$4: now also S1.13; no longer 1-10VPP.1
- net N$40: now also S1.4; no longer 1-10VPP.8
- net N$41: now also S1.3; no longer 1-10VPP.7
- net N$44: now also S1.15; no longer 1-10VPP.3
- net N$45: now also S1.16; no longer 1-10VPP.4
- net N$5: now also S1.14; no longer 1-10VPP.2
- net VPWR: now also L4.P$1, R93.2, R95.2; no longer C32.1, D1.C, D14.C, D2.C, U3.1, U3.3
